File: CISYNTH.sch (KiCad schematic (older format))
At the start: 142 parts, among them K1 BATT, K10 TOF_RD, K11 TOF_RS, K12 TOF_LF, K13 TOF_LD, K14 TOF_LS, K2 K_FPC_52435-2471, K3 DVB_JTAG-10, K5 K_PicoSPOX-3, K6 K_0002, K7 K_PicoSPOX-3, K8 K_0002, K9 TOF_RF, Q1 Q_0004, Q2 Q_0007, Q3 Q_0007, Q4 Q_0007, Q5 Q_0007, Q6 Q_0007, Q7 Q_0007, Q8 Q_0004, Q9 Q_0004, SW1 SW_SKQG, SW2 SW_SKQG, U1 U_LT8610ABIMSE-3.3, U10 QRE1113GR, U11 QRE1113GR, U12 QRE1113GR, U2 U_AP2204K-5.0TRG1, U3 LTC2944, U4 L6234, U5 L6234, U6 LTC2955TS8-1, U7 STM32H743VITx, U8 ICM-20689, U9 QRE1113GR

Commit message: Daftpink
Parts:
- added SW?: Rotary_Encoder_Switch, symbol Rotary_Encoder_Switch
Changed lines of the file:
@@
 LIBS:DVB_XO
 LIBS:nara
-LIBS:NARA-cache
+LIBS:Video
+LIBS:Valve
+LIBS:Triac_Thyristor
+LIBS:Transistor_IGBT
+LIBS:Transistor_FET
+LIBS:Transistor_BJT
+LIBS:Transistor_Array
+LIBS:Transformer
+LIBS:Timer_RTC
+LIBS:Timer_PLL
+LIBS:Timer
+LIBS:Switch
+LIBS:Sensor_Voltage
+LIBS:Sensor_Touch
+LIBS:Sensor_Temperature
+LIBS:Sensor_Proximity
+LIBS:Sensor_Pressure
+LIBS:Sensor_Optical
+LIBS:Sensor_Motion
+LIBS:Sensor_Magnetic
+LIBS:Sensor_Humidity
+LIBS:Sensor_Gas
+LIBS:Sensor_Current
+LIBS:Sensor_Audio
+LIBS:Sensor
+LIBS:RF_ZigBee
+LIBS:RF_WiFi
+LIBS:RF_Switch
+LIBS:RF_RFID
+LIBS:RF_Module
+LIBS:RF_Mixer
+LIBS:RF_GPS
+LIBS:RF_Bluetooth
+LIBS:RF_Amplifier
+LIBS:RF_AM_FM
+LIBS:RF
+LIBS:Relay_SolidState
+LIBS:Relay
+LIBS:Regulator_Switching
+LIBS:Regulator_SwitchedCapacitor
+LIBS:Regulator_Linear
+LIBS:Regulator_Current
+LIBS:Regulator_Controller
+LIBS:Reference_Voltage
+LIBS:Reference_Current
+LIBS:pspice
+LIBS:Power_Supervisor
+LIBS:Power_Protection
+LIBS:Power_Management
+LIBS:power
+LIBS:Potentiometer_Digital
+LIBS:Oscillator
+LIBS:Motor
+LIBS:Memory_UniqueID
+LIBS:Memory_ROM
+LIBS:Memory_RAM
+LIBS:Memory_NVRAM
+LIBS:Memory_Flash
+LIBS:Memory_EPROM
+LIBS:Memory_EEPROM
+LIBS:Memory_Controller
+LIBS:Mechanical
+LIBS:MCU_Texas_MSP430
+LIBS:MCU_Texas
+LIBS:MCU_ST_STM32L4+
+LIBS:MCU_ST_STM32L4
+LIBS:MCU_ST_STM32L1
+LIBS:MCU_ST_STM32L0
+LIBS:MCU_ST_STM32H7
+LIBS:MCU_ST_STM32F7
+LIBS:MCU_ST_STM32F4
+LIBS:MCU_ST_STM32F3
+LIBS:MCU_ST_STM32F2
+LIBS:MCU_ST_STM32F1
+LIBS:MCU_ST_STM32F0
+LIBS:MCU_ST_STM8
+LIBS:MCU_SiliconLabs
+LIBS:MCU_SiFive
+LIBS:MCU_Parallax
+LIBS:MCU_NXP_S08
+LIBS:MCU_NXP_MCore
+LIBS:MCU_NXP_MAC7100
+LIBS:MCU_NXP_LPC
+LIBS:MCU_NXP_Kinetis
+LIBS:MCU_NXP_HCS12
+LIBS:MCU_NXP_HC12
+LIBS:MCU_NXP_HC11
+LIBS:MCU_NXP_ColdFire
+LIBS:MCU_Nordic
+LIBS:MCU_Module
+LIBS:MCU_Microchip_SAML
+LIBS:MCU_Microchip_SAME
+LIBS:MCU_Microchip_PIC32
+LIBS:MCU_Microchip_PIC24
+LIBS:MCU_Microchip_PIC18
+LIBS:MCU_Microchip_PIC16
+LIBS:MCU_Microchip_PIC12
+LIBS:MCU_Microchip_PIC10
+LIBS:MCU_Microchip_AVR
+LIBS:MCU_Microchip_ATtiny
+LIBS:MCU_Microchip_ATmega
+LIBS:MCU_Microchip_8051
+LIBS:MCU_Intel
+LIBS:MCU_Espressif
+LIBS:MCU_Cypress
+LIBS:MCU_AnalogDevices
+LIBS:Logic_Programmable
+LIBS:Logic_LevelTranslator
+LIBS:LED
+LIBS:Jumper
+LIBS:Isolator_Analog
+LIBS:Isolator
+LIBS:Interface_USB
+LIBS:Interface_UART
+LIBS:Interface_Telecom
+LIBS:Interface_Optical
+LIBS:Interface_LineDriver
+LIBS:Interface_HID
+LIBS:Interface_Expansion
+LIBS:Interface_Ethernet
+LIBS:Interface_CurrentLoop
+LIBS:Interface_CAN_LIN
+LIBS:Interface
+LIBS:Graphic
+LIBS:GPU
+LIBS:FPGA_Xilinx_Virtex7
+LIBS:FPGA_Xilinx_Virtex6
+LIBS:FPGA_Xilinx_Virtex5
+LIBS:FPGA_Xilinx_Spartan6
+LIBS:FPGA_Xilinx_Kintex7
+LIBS:FPGA_Xilinx_Artix7
+LIBS:FPGA_Xilinx
+LIBS:FPGA_Microsemi
+LIBS:Filter
+LIBS:DSP_Texas
+LIBS:DSP_Motorola
+LIBS:DSP_Microchip_DSPIC33
+LIBS:DSP_Freescale
+LIBS:Driver_Relay
+LIBS:Driver_Motor
+LIBS:Driver_LED
+LIBS:Driver_FET
+LIBS:Driver_Display
+LIBS:Display_Graphic
+LIBS:Display_Character
+LIBS:Diode_Laser
+LIBS:Diode_Bridge
+LIBS:Diode
+LIBS:Device
+LIBS:CPU_PowerPC
+LIBS:CPU_NXP_68000
+LIBS:CPU_NXP_6800
+LIBS:CPU
+LIBS:CPLD_Xilinx
+LIBS:CPLD_Altera
+LIBS:Converter_DCDC
+LIBS:Converter_ACDC
+LIBS:Connector_Generic_Shielded
+LIBS:Connector_Generic_MountingPin
+LIBS:Connector_Generic
+LIBS:Connector
+LIBS:Comparator
+LIBS:Battery_Management
+LIBS:Audio
+LIBS:Analog_Switch
+LIBS:Analog_DAC
+LIBS:Analog_ADC
+LIBS:Analog
+LIBS:Amplifier_Video
+LIBS:Amplifier_Operational
+LIBS:Amplifier_Instrumentation
+LIBS:Amplifier_Difference
+LIBS:Amplifier_Current
+LIBS:Amplifier_Buffer
+LIBS:Amplifier_Audio
+LIBS:74xx_IEEE
+LIBS:74xx
+LIBS:74xGxx
+LIBS:4xxx_IEEE
+LIBS:4xxx
+LIBS:CISYNTH-cache
 EELAYER 25 0
 EELAYER END
@@
 Text Label 9050 4450 2    60   ~ 0
 MOT_L_IN3
+$Comp
+L Rotary_Encoder_Switch SW?
+U 1 1 5B1F050B
+P 4650 4875
+F 0 "SW?" H 4650 5135 50  0000 C CNN
+F 1 "Rotary_Encoder_Switch" H 4650 4615 50  0000 C CNN
+F 2 "" H 4500 5035 50  0001 C CNN
+F 3 "" H 4650 5135 50  0001 C CNN
+	1    4650 4875
+	1    0    0    -1
+$EndComp
 $EndSCHEMATC

Commit message: Update project
Parts:
- removed K1: BATT, NARA_Lib:Pin_Header_Straight_1x02_Pitch3mm, symbol CONN_01X02
- removed R8: R_0002, DVB_Resistors:R_0402, symbol R_0002
- added A1: Pololu_DRV8825, Module:Pololu_Breakout-16_15.2x20.3mm, symbol Pololu_Breakout_DRV8825
- added C20: C_0058, DVB_Capacitors_Tantalum:CP_EIA-7343-31, symbol C_0058
- added C27: C_0002, DVB_Capacitors_Ceramic:C_0402, symbol C_0002
- added C32, C46: C_0040, DVB_Capacitors_Ceramic:C_1210, symbol C_0040
- added J1: Jack-DC, Connectors:BARREL_JACK, symbol Jack-DC
- added J2: USB_B_Mini, Connector_USB:USB_Mini-B_Lumberg_2486_01_Horizontal, symbol USB_B_Mini
- added J3: AudioJack3_Switch, CISYNTH_Lib:Connector_Amphenol, symbol AudioJack3_Switch
- added J4: MOTOR, symbol Screw_Terminal_01x04
- added J5: LIMIT_SWITCH, symbol Screw_Terminal_01x02
- added J6: VIDEO_OUT, Connector_Dsub:DSUB-15-HD_Female_Horizontal_P2.29x1.98mm_EdgePinOffset8.35mm_Housed_MountingHolesOffset10.89mm, symbol DB15_Female_HighDensity_MountingHoles
- added J7: CIS_FPC, Connector_FFC-FPC:TE_1-84953-2_1x12-1MP_P1.0mm_Horizontal, symbol Conn_01x12
- added Q10, Q12, Q14: PMST3904, DVB_SOT:SOT_23, symbol Q_NPN_BEC
- added Q11, Q13, Q15: PDTC143EU, DVB_SOT:SOT_23, symbol Q_NPN_BEC
- added R20, R59: R_0020, DVB_Resistors:R_0402, symbol R_0020
- added R21, R22, R24: R, DVB_Resistors:R_0402, symbol R
- added R25, R26, R27: R_0033, DVB_Resistors:R_0402, symbol R_0033
- added R28, R51, R52: R, DVB_Resistors:R_0603, symbol R
- added R58: R_0015, DVB_Resistors:R_0402, symbol R_0015
- added R8, R? (x6): R, n.c, symbol R
- added RV1, RV?: R_POT, Potentiometers:Potentiometer_Alps_RK09K_Horizontal, symbol R_POT
- added SW4: Rotary_Encoder_Switch, Rotary_Encoder:RotaryEncoder_Alps_EC11E-Switch_Vertical_H20mm, symbol Rotary_Encoder_Switch
- added U13: LM324, Package_SO:SOIC-14_3.9x8.7mm_P1.27mm, symbol LM324
- SW3: renamed from SW?; footprint (none) -> Rotary_Encoder:RotaryEncoder_Alps_EC11E-Switch_Vertical_H20mm
Connections:
- net labels added: +12V, CIS_CLK, CIS_LED_B, CIS_LED_G, CIS_LED_R, CIS_SP, CIS_VREF_HI, CIS_VREF_LO, LED_BLUE, LED_GREEN, LED_RED, MOTOR_DIR, MOTOR_EN, MOTOR_M0, MOTOR_M1, MOTOR_M2, MOTOR_STEP, VGA_BLUE, VGA_BLUE_1, VGA_BLUE_2, VGA_GREEN, VGA_GREEN_1, VGA_GREEN_2, VGA_H_SYNC, VGA_ID0/RES, VGA_ID1/SDA, VGA_ID2/RES, VGA_ID3/SCL, VGA_KEY/PWR, VGA_RED, VGA_RED_1, VGA_RED_2, VGA_V_SYNC, VREF_LO
- wire segments 161 -> 221
- no-connect marks 28 -> 5
Other:
- note added: "VERIFIER PINNOUT (SENS)"
