File: CIS/CIS.sch (KiCad schematic (older format))
At the start: 181 parts, among them J1 Conn_01x12, J2 RJ45_Abracon_ARJP11A-MASA-B-A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, J3 SJ1-3533NG, J4 DEBUG TAG, K1 K_9999, P3 K_0023, Q1 Q_0002, Q2 Q_0002, Q3 Q_0002, SW1 SW_0003, SW2 SW_0003, SW3 SW_0003, SW4 SW_0003, SW5 SW_0003, U1 U_0076, U14 U_0101, U16 U_0049, U17 U_0049, U2 STM32H745IIKx, U3 U_0103, U4 U_1001, U5 U_0081, U6 U_0097, U7 PCM5102, U8 ICM-20602

Commit message: Incert CIS connector
Parts:
- removed J1: Conn_01x12, DVB_Connectors:Molex_PicoBlade_53048-1210_1x12_P1.25mm_Horizontal, symbol Connector_Generic:Conn_01x12
- added J1: K_9998, DVB_Connectors:Molex_PicoBlade_53261-1271_1x12-1MP_P1.25mm_Horizontal, symbol DVB_K:K_9998
Connections:
- net +5V: now also J1.4 (Pin_4), J1.8 (Pin_8)
- net CIS_CP: now also U6.4 (A3); no longer U6.2 (A1)
- net CIS_CP_TTL: now also U6.11 (B3); no longer U6.13 (B1)
- net CIS_LED_B: now also U2.E14 (PC6); no longer U2.N15 (PH12)
- net CIS_LED_G: now also U2.N15 (PH12); no longer U2.H15 (PD13)
- net CIS_LED_R: now also U2.H15 (PD13); no longer U2.E14 (PC6)
- net CIS_RS: now also U6.2 (A1); no longer U6.5 (A4)
- net CIS_RS_TTL: now also U6.13 (B1), J1.9 (Pin_9); no longer U6.10 (B4)
- net CIS_SP_TTL: now also J1.7 (Pin_7)
- net CIS_VLED_B: now also J1.1 (Pin_1)
- net CIS_VLED_G: now also J1.3 (Pin_3)
- net CIS_VLED_R: now also J1.2 (Pin_2)
- net GND: now also J1.6 (Pin_6)
- net at R12.2: now also J1.12 (Pin_12)
- net at R13.2: now also J1.11 (Pin_11)
- net at R14.2: now also J1.10 (Pin_10)
- net at C37.2, R15.1: now also J1.5 (Pin_5)
Other:
- note added: "150mm Molex cable : 0151341202‎"
Changed lines of the file:
@@
 	1    0    0    -1
 $EndComp
-Text Label 4475 4150 2    39   ~ 0
+Text Label 4475 4350 2    39   ~ 0
 CIS_CP
 Text Label 6800 2825 1    39   ~ 0
@@
 $EndComp
 Connection ~ 4550 7475
-Text Label 5475 4450 0    39   ~ 0
+Text Label 5475 4150 0    39   ~ 0
 CIS_RS_TTL
 Text Label 5475 4250 0    39   ~ 0
@@
 	0    1    1    0
 $EndComp
-NoConn ~ 5475 4350
 Text Label 4475 4250 2    39   ~ 0
 CIS_SP
-Text Label 5475 4150 0    39   ~ 0
+Text Label 5475 4350 0    39   ~ 0
 CIS_CP_TTL
-Text Label 4475 4450 2    39   ~ 0
+Text Label 4475 4150 2    39   ~ 0
 CIS_RS
-NoConn ~ 4475 4350
 $Comp
 L CIS-rescue:+3.3V-HM3-rescue #PWR0228
@@
 Text Label 4125 2750 2    39   ~ 0
 CIS_ADC_3
-$Comp
-L Connector_Generic:Conn_01x12 J1
-U 1 1 60501103
-P 5275 2550
-F 0 "J1" H 5275 3150 50  0000 C CNN
-F 1 "Conn_01x12" V 5375 2500 50  0000 C CNN
-F 2 "DVB_Connectors:Molex_PicoBlade_53048-1210_1x12_P1.25mm_Horizontal" H 5275 2550 50  0001 C CNN
-F 3 "~" H 5275 2550 50  0001 C CNN
-	1    5275 2550
-	0    -1   -1   0
-$EndComp
 $Comp
 L DVB_R:R_0134 R15
@@
 Text Label 20400 6725 0    39   ~ 0
 RMII_RXD0
-Text Label 20400 6825 0    39   ~ 0
-RMII_RXD1
 Text Label 20400 6225 0    39   ~ 0
 RMII_MDC
@@
 	0    -1   1    0
 $EndComp
+Text Label 20400 9325 0    39   ~ 0
+CIS_LED_R
+Text Label 15650 5025 2    39   ~ 0
+CIS_LED_G
+Text Notes 4500 2300 0    60   ~ 0
+150mm Molex cable : 0151341202‎
+$Comp
+L DVB_K:K_9998 J1
+U 1 1 5FF53592
+P 5375 2550
+F 0 "J1" H 5375 3150 50  0000 C CNN
+F 1 "K_9998" V 5725 2550 50  0001 C CNN
+F 2 "DVB_Connectors:Molex_PicoBlade_53261-1271_1x12-1MP_P1.25mm_Horizontal" V 5625 2550 50  0001 C CNN
+F 3 "https://www.molex.com/pdm_docs/sd/532611271_sd.pdf" H 5375 2550 50  0001 C CNN
+F 4 "532611271" V 5475 2550 50  0000 C CNN "Field4"
+	1    5375 2550
+	0    1    -1   0
+$EndComp
+NoConn ~ 5475 4450
+NoConn ~ 4475 4450
 Text Label 20400 6925 0    39   ~ 0
-CIS_LED_R
-Text Label 20400 9325 0    39   ~ 0
-CIS_LED_G
-Text Label 15650 5025 2    39   ~ 0
 CIS_LED_B
+Text Label 20400 6825 0    39   ~ 0
+RMII_RXD1
 $EndSCHEMATC
