File: CIS/CIS.kicad_pcb (KiCad board)
At the start: 6 copper layers, 122 x 32.5 mm, 189 parts, among them J1 K_9998, J2 RJ45_Abracon_ARJP11A-MASA-B-A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, J3 SJ1-3533NG, J4 DEBUG TAG, K1 K_9999, P3 K_0023, Q1 Q_0002, Q2 Q_0002, Q3 Q_0002, SW1 SW_0003, SW2 SW_0003, SW3 SW_0003, SW4 SW_0003, SW5 SW_0003, U1 U_0076, U14 U_0101, U16 U_0049, U17 U_0049, U2 STM32H745IIKx, U3 U_0103, U4 U_1001, U5 U_0081, U6 U_0097, U7 PCM5102, U8 ICM-20602

Commit message: move buttons
Parts:
- moved R26 4.10 mm to (152.3, 100.6)
- moved R42 4.10 mm to (152.3, 101.8)
- moved C53 4.10 mm to (152.1, 99.4)
- moved SW3 4.10 mm to (156.2, 101.7)
- moved R18 3.35 mm to (163.6, 100.6)
- moved R21 3.35 mm to (163.6, 101.8)
- moved C40 3.35 mm to (163.3, 99.4)
- moved SW1 3.35 mm to (167.4, 101.7)
- moved R45 2.60 mm to (174.8, 100.6)
- moved R46 2.60 mm to (174.8, 101.8)
- moved C57 2.60 mm to (174.6, 99.4)
- moved SW5 2.60 mm to (178.7, 101.7)
- moved R19 1.85 mm to (186.1, 100.6)
- moved R22 1.85 mm to (186.1, 101.8)
- moved C42 1.85 mm to (185.8, 99.4)
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Routing:
- net GND: track 125.4 -> 130.3 mm, vias 142 -> 143
- net /12V_EN: track 24.5 -> 27.3 mm
- net +3.3V: track 72.1 -> 74.9 mm, vias 49 -> 50
- net /SW_OK: track 25.9 -> 28.5 mm
- net /SW_RIGHT: track 30.8 -> 28.9 mm
- net /SWD-CLK: track 39.7 -> 38.4 mm
- net /SW_DOWN: track 37.6 -> 38.7 mm
- net /SW_UP: track 25.9 -> 26.8 mm
- net Net-(C44-Pad1): vias 4 -> 7
- added copper zone on In1.Cu, net Net-(C44-Pad1)
